File: custom-mech.sch (KiCad schematic (older format))
At the start: 161 parts

Commit message: added footprints
Parts:
- C1, C2, C3, C4, C5, C6, C7: renamed from C?; footprint (none) -> Capacitor_SMD:C_0805_2012Metric
- D1, D10, D11, D12, D13, D14, D15, D16, D17, D18, D19, D2, D20, D21, D22, D23, D24, D25, D26, D27, D28, D29, D3, D30, D31, D32, D33, D34, D35, D36, D37, D38, D39, D4, D40, D41, D42, D43, D44, D45, D46, D47, D48, D49, D5, D50, D51, D52, D53, D54, D55, D56, D57, D58, D59, D6, D60, D61, D62, D63, D64, D65, D66, D67, D68, D69, D7, D70, D8, D9: renamed from D?; footprint (none) -> Diode_SMD:D_SOD-123
- F1: renamed from F?; footprint (none) -> Fuse:Fuse_1206_3216Metric
- MX1, MX10, MX11, MX12, MX13, MX14, MX15, MX16, MX17, MX18, MX19, MX2, MX20, MX21, MX22, MX23, MX24, MX25, MX26, MX27, MX28, MX29, MX3, MX30, MX31, MX32, MX33, MX34, MX35, MX36, MX37, MX38, MX39, MX4, MX40, MX41, MX42, MX43, MX44, MX45, MX46, MX47, MX48, MX49, MX5, MX50, MX51, MX52, MX53, MX54, MX55, MX56, MX57, MX58, MX59, MX6, MX60, MX61, MX62, MX63, MX64, MX65, MX66, MX67, MX68, MX69, MX7, MX70, MX71, MX72, MX73, MX74, MX75, MX8, MX9: renamed from MX?; footprint (none) -> Button_Switch_Keyboard:SW_Cherry_MX_1.00u_PCB
- R1, R2, R3, R4: renamed from R?; footprint (none) -> Resistor_SMD:R_0805_2012Metric
- SW1: renamed from SW?; footprint (none) -> random-keyboard-parts:SKQG-1155865
- USB1: renamed from USB?; footprint (none) -> random-keyboard-parts:Molex-0548190589
- Y1: renamed from Y?; footprint (none) -> Crystal:Crystal_SMD_3225-4Pin_3.2x2.5mm
- gave numbers to parts that had none: 1

Commit message: saved lol
Connections:
- net labels added: COL0, COL1, COL10, COL11, COL12, COL13, COL2, COL3, COL4, COL5, COL6, COL7, COL8, COL9, ROW2, ROW3, ROW4
- wire segments 254 -> 255
Changed lines of the file:
@@
 	1900 -2300 1600 -2300
 Text GLabel 1600 -2300 0    50   Input ~ 0
-ROW1
+ROW2
 $Comp
 L MX_Alps_Hybrid:MX-NoLED MX33
@@
 	1900 -1700 1600 -1700
 Text GLabel 1600 -1700 0    50   Input ~ 0
-ROW1
+ROW3
 $Comp
 L MX_Alps_Hybrid:MX-NoLED MX48
@@
 	1900 -1100 1600 -1100
 Text GLabel 1600 -1100 0    50   Input ~ 0
-ROW1
+ROW4
 $Comp
 L MX_Alps_Hybrid:MX-NoLED MX63
@@
 Wire Wire Line
 	9700 -1100 9100 -1100
+Text GLabel -500 -3500 2    50   Input ~ 0
+D-
+Text GLabel -500 -3400 2    50   Input ~ 0
+D+
+$Comp
+L power:GND #PWR?
+U 1 1 607822F8
+P -400 -3200
+F 0 "#PWR?" H -400 -3450 50  0001 C CNN
+F 1 "GND" H -395 -3373 50  0000 C CNN
+F 2 "" H -400 -3200 50  0001 C CNN
+F 3 "" H -400 -3200 50  0001 C CNN
+	1    -400 -3200
+	1    0    0    -1
+$EndComp
+Wire Wire Line
+	-500 -3200 -400 -3200
+Text GLabel 2250 -4200 1    50   Input ~ 0
+COL0
+Text GLabel 2850 -4200 1    50   Input ~ 0
+COL1
+Text GLabel 3450 -4200 1    50   Input ~ 0
+COL2
+Text GLabel 4050 -4200 1    50   Input ~ 0
+COL3
+Text GLabel 4650 -4200 1    50   Input ~ 0
+COL4
+Text GLabel 5250 -4200 1    50   Input ~ 0
+COL5
+Text GLabel 5850 -4200 1    50   Input ~ 0
+COL6
+Text GLabel 6450 -4200 1    50   Input ~ 0
+COL7
+Text GLabel 7050 -4200 1    50   Input ~ 0
+COL8
+Text GLabel 7650 -4200 1    50   Input ~ 0
+COL9
+Text GLabel 8250 -4200 1    50   Input ~ 0
+COL10
+Text GLabel 8850 -4200 1    50   Input ~ 0
+COL11
+Text GLabel 9450 -4200 1    50   Input ~ 0
+COL12
+Text GLabel 10050 -4200 1    50   Input ~ 0
+COL13
 $EndSCHEMATC

Commit message: finished pcb
Parts:
- removed MX24, MX39, MX54, MX69, MX9: MX-NoLED, Button_Switch_Keyboard:SW_Cherry_MX_1.00u_PCB, symbol MX_Alps_Hybrid:MX-NoLED
- MX1, MX2, MX3, MX4, MX5, MX6, MX7, MX8: footprint Button_Switch_Keyboard:SW_Cherry_MX_1.00u_PCB -> MX_Alps_Hybrid:MX-1U
- MX10: renamed from MX11; footprint Button_Switch_Keyboard:SW_Cherry_MX_1.00u_PCB -> MX_Alps_Hybrid:MX-1U
- MX11: renamed from MX12; footprint Button_Switch_Keyboard:SW_Cherry_MX_1.00u_PCB -> MX_Alps_Hybrid:MX-1U
- MX12: renamed from MX13; footprint Button_Switch_Keyboard:SW_Cherry_MX_1.00u_PCB -> MX_Alps_Hybrid:MX-1U
- MX13: renamed from MX14; footprint Button_Switch_Keyboard:SW_Cherry_MX_1.00u_PCB -> MX_Alps_Hybrid:MX-1U
- MX14: renamed from MX15; footprint Button_Switch_Keyboard:SW_Cherry_MX_1.00u_PCB -> MX_Alps_Hybrid:MX-1U
- MX15: renamed from MX16; footprint Button_Switch_Keyboard:SW_Cherry_MX_1.00u_PCB -> MX_Alps_Hybrid:MX-1U
- MX16: renamed from MX17; footprint Button_Switch_Keyboard:SW_Cherry_MX_1.00u_PCB -> MX_Alps_Hybrid:MX-1U
- MX17: renamed from MX18; footprint Button_Switch_Keyboard:SW_Cherry_MX_1.00u_PCB -> MX_Alps_Hybrid:MX-1U
- MX18: renamed from MX19; footprint Button_Switch_Keyboard:SW_Cherry_MX_1.00u_PCB -> MX_Alps_Hybrid:MX-1U
- MX19: renamed from MX20; footprint Button_Switch_Keyboard:SW_Cherry_MX_1.00u_PCB -> MX_Alps_Hybrid:MX-1U
- MX20: renamed from MX21; footprint Button_Switch_Keyboard:SW_Cherry_MX_1.00u_PCB -> MX_Alps_Hybrid:MX-1U
- MX21: renamed from MX22; footprint Button_Switch_Keyboard:SW_Cherry_MX_1.00u_PCB -> MX_Alps_Hybrid:MX-1U
- MX22: renamed from MX23; footprint Button_Switch_Keyboard:SW_Cherry_MX_1.00u_PCB -> MX_Alps_Hybrid:MX-1U
- MX23: renamed from MX25; footprint Button_Switch_Keyboard:SW_Cherry_MX_1.00u_PCB -> MX_Alps_Hybrid:MX-1U
- MX24: renamed from MX26; footprint Button_Switch_Keyboard:SW_Cherry_MX_1.00u_PCB -> MX_Alps_Hybrid:MX-1U
- MX25: renamed from MX27; footprint Button_Switch_Keyboard:SW_Cherry_MX_1.00u_PCB -> MX_Alps_Hybrid:MX-1U
- MX26: renamed from MX28; footprint Button_Switch_Keyboard:SW_Cherry_MX_1.00u_PCB -> MX_Alps_Hybrid:MX-1U
- MX27: renamed from MX29; footprint Button_Switch_Keyboard:SW_Cherry_MX_1.00u_PCB -> MX_Alps_Hybrid:MX-1U
- MX28: renamed from MX30; footprint Button_Switch_Keyboard:SW_Cherry_MX_1.00u_PCB -> MX_Alps_Hybrid:MX-1U
- MX29: renamed from MX31; footprint Button_Switch_Keyboard:SW_Cherry_MX_1.00u_PCB -> MX_Alps_Hybrid:MX-1U
- MX30: renamed from MX32; footprint Button_Switch_Keyboard:SW_Cherry_MX_1.00u_PCB -> MX_Alps_Hybrid:MX-1U
- MX31: renamed from MX33; footprint Button_Switch_Keyboard:SW_Cherry_MX_1.00u_PCB -> MX_Alps_Hybrid:MX-1U
- MX32: renamed from MX34; footprint Button_Switch_Keyboard:SW_Cherry_MX_1.00u_PCB -> MX_Alps_Hybrid:MX-1U
- MX33: renamed from MX35; footprint Button_Switch_Keyboard:SW_Cherry_MX_1.00u_PCB -> MX_Alps_Hybrid:MX-1U
- MX34: renamed from MX36; footprint Button_Switch_Keyboard:SW_Cherry_MX_1.00u_PCB -> MX_Alps_Hybrid:MX-1U
- MX35: renamed from MX37; footprint Button_Switch_Keyboard:SW_Cherry_MX_1.00u_PCB -> MX_Alps_Hybrid:MX-1U
- MX36: renamed from MX38; footprint Button_Switch_Keyboard:SW_Cherry_MX_1.00u_PCB -> MX_Alps_Hybrid:MX-1U
- MX37: renamed from MX40; footprint Button_Switch_Keyboard:SW_Cherry_MX_1.00u_PCB -> MX_Alps_Hybrid:MX-1U
- MX38: renamed from MX41; footprint Button_Switch_Keyboard:SW_Cherry_MX_1.00u_PCB -> MX_Alps_Hybrid:MX-1U
- MX39: renamed from MX42; footprint Button_Switch_Keyboard:SW_Cherry_MX_1.00u_PCB -> MX_Alps_Hybrid:MX-1U
- MX40: renamed from MX43; footprint Button_Switch_Keyboard:SW_Cherry_MX_1.00u_PCB -> MX_Alps_Hybrid:MX-1U
- MX41: renamed from MX44; footprint Button_Switch_Keyboard:SW_Cherry_MX_1.00u_PCB -> MX_Alps_Hybrid:MX-1U
- MX42: renamed from MX45; footprint Button_Switch_Keyboard:SW_Cherry_MX_1.00u_PCB -> MX_Alps_Hybrid:MX-1U
- MX43: renamed from MX46; footprint Button_Switch_Keyboard:SW_Cherry_MX_1.00u_PCB -> MX_Alps_Hybrid:MX-1U
- MX44: renamed from MX47; footprint Button_Switch_Keyboard:SW_Cherry_MX_1.00u_PCB -> MX_Alps_Hybrid:MX-1U
- MX45: renamed from MX48; footprint Button_Switch_Keyboard:SW_Cherry_MX_1.00u_PCB -> MX_Alps_Hybrid:MX-1U
- MX46: renamed from MX49; footprint Button_Switch_Keyboard:SW_Cherry_MX_1.00u_PCB -> MX_Alps_Hybrid:MX-1U
- MX47: renamed from MX50; footprint Button_Switch_Keyboard:SW_Cherry_MX_1.00u_PCB -> MX_Alps_Hybrid:MX-1U
- MX48: renamed from MX51; footprint Button_Switch_Keyboard:SW_Cherry_MX_1.00u_PCB -> MX_Alps_Hybrid:MX-1U
- MX49: renamed from MX52; footprint Button_Switch_Keyboard:SW_Cherry_MX_1.00u_PCB -> MX_Alps_Hybrid:MX-1U
- MX50: renamed from MX53; footprint Button_Switch_Keyboard:SW_Cherry_MX_1.00u_PCB -> MX_Alps_Hybrid:MX-1U
- MX51: renamed from MX55; footprint Button_Switch_Keyboard:SW_Cherry_MX_1.00u_PCB -> MX_Alps_Hybrid:MX-1U
- MX52: renamed from MX56; footprint Button_Switch_Keyboard:SW_Cherry_MX_1.00u_PCB -> MX_Alps_Hybrid:MX-1U
- MX53: renamed from MX57; footprint Button_Switch_Keyboard:SW_Cherry_MX_1.00u_PCB -> MX_Alps_Hybrid:MX-1U
- MX54: renamed from MX58; footprint Button_Switch_Keyboard:SW_Cherry_MX_1.00u_PCB -> MX_Alps_Hybrid:MX-1U
- MX55: renamed from MX59; footprint Button_Switch_Keyboard:SW_Cherry_MX_1.00u_PCB -> MX_Alps_Hybrid:MX-1U
- MX56: renamed from MX60; footprint Button_Switch_Keyboard:SW_Cherry_MX_1.00u_PCB -> MX_Alps_Hybrid:MX-1U
- MX57: renamed from MX61; footprint Button_Switch_Keyboard:SW_Cherry_MX_1.00u_PCB -> MX_Alps_Hybrid:MX-1U
- MX58: renamed from MX62; footprint Button_Switch_Keyboard:SW_Cherry_MX_1.00u_PCB -> MX_Alps_Hybrid:MX-1U
- MX59: renamed from MX63; footprint Button_Switch_Keyboard:SW_Cherry_MX_1.00u_PCB -> MX_Alps_Hybrid:MX-1U
- MX60: renamed from MX64; footprint Button_Switch_Keyboard:SW_Cherry_MX_1.00u_PCB -> MX_Alps_Hybrid:MX-1U
- MX61: renamed from MX65; footprint Button_Switch_Keyboard:SW_Cherry_MX_1.00u_PCB -> MX_Alps_Hybrid:MX-1U
- MX62: renamed from MX66; footprint Button_Switch_Keyboard:SW_Cherry_MX_1.00u_PCB -> MX_Alps_Hybrid:MX-1U
- MX63: renamed from MX67; footprint Button_Switch_Keyboard:SW_Cherry_MX_1.00u_PCB -> MX_Alps_Hybrid:MX-1U
- MX64: renamed from MX68; footprint Button_Switch_Keyboard:SW_Cherry_MX_1.00u_PCB -> MX_Alps_Hybrid:MX-1U
- MX65: renamed from MX70; footprint Button_Switch_Keyboard:SW_Cherry_MX_1.00u_PCB -> MX_Alps_Hybrid:MX-1U
- MX66: renamed from MX71; footprint Button_Switch_Keyboard:SW_Cherry_MX_1.00u_PCB -> MX_Alps_Hybrid:MX-1U
- MX67: renamed from MX72; footprint Button_Switch_Keyboard:SW_Cherry_MX_1.00u_PCB -> MX_Alps_Hybrid:MX-1U
- MX68: renamed from MX73; footprint Button_Switch_Keyboard:SW_Cherry_MX_1.00u_PCB -> MX_Alps_Hybrid:MX-1U
- MX69: renamed from MX74; footprint Button_Switch_Keyboard:SW_Cherry_MX_1.00u_PCB -> MX_Alps_Hybrid:MX-1U
- MX70: renamed from MX75; footprint Button_Switch_Keyboard:SW_Cherry_MX_1.00u_PCB -> MX_Alps_Hybrid:MX-1U
- MX9: renamed from MX10; footprint Button_Switch_Keyboard:SW_Cherry_MX_1.00u_PCB -> MX_Alps_Hybrid:MX-1U
Connections:
- net COL0: now also U1.30 (PB6)
- net COL1: now also U1.31 (PC6)
- net COL10: now also U1.19 (PD1)
- net COL11: now also U1.20 (PD2)
- net COL12: now also U1.21 (PD3)
- net COL13: now also U1.22 (PD5)
- net COL2: now also U1.32 (PC7)
- net COL3: now also U1.36 (PF7)
- net COL4: now also U1.37 (PF6)
- net COL5: now also U1.38 (PF5)
- net COL6: now also U1.39 (PF4)
- net COL7: now also U1.40 (PF1)
- net COL8: now also U1.41 (PF0)
- net COL9: now also U1.18 (PD0)
- net ROW0: now also U1.25 (PD4)
- net ROW1: now also U1.26 (PD6)
- net ROW2: now also U1.27 (PD7)
- net ROW3: now also U1.28 (PB4)
- net ROW4: now also U1.29 (PB5)
Other:
- moved on the sheet: F1, USB1
