File: atmega/custom-mech atmega.kicad_pcb (KiCad board)
At the start: 2 copper layers, 292.9 x 97.5 mm, 156 parts, among them SW1 SW_Push, U1 ATmega32U4-AU, Y1 16MHz

Commit message: small updates
Parts:
- moved C1 365.8 mm to (63.9, 105.4)
- moved C2 365.8 mm to (55.1, 105.4)
- moved C3 365.8 mm to (50.2, 119.4)
- moved C4 365.8 mm to (50.2, 109.1)
- moved C7 365.8 mm to (68.3, 112.5)
- moved D15 365.8 mm to (88.2, 65.6)
- moved D16 365.8 mm to (107.2, 65.6)
- moved D17 365.8 mm to (126.3, 65.6)
- moved D18 365.8 mm to (145.3, 65.6)
- moved D19 365.8 mm to (164.4, 65.6)
- moved D20 365.8 mm to (183.4, 65.6)
- moved D21 365.8 mm to (202.5, 65.6)
- moved D22 365.8 mm to (221.5, 65.6)
- moved D23 365.8 mm to (240.6, 65.6)
- moved D24 365.8 mm to (259.6, 65.6)
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