File: atmega/custom-mech.sch (KiCad schematic (older format))
At the start: 156 parts, among them SW1 SW_Push, U1 ATmega32U4-AU, Y1 16MHz

Commit message: small updates
Other:
- moved on the sheet: C1, C2, C3, C4, C5, C6, C7, D1, D10, D11, D12, D13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
