File: pro micro version/pro micro version new traces.kicad_pcb (KiCad board)
At the start: 2 copper layers, 385.8 x 100 mm, 166 parts, among them SW1 SW_PUSH, U1 ProMicro

Commit message: autosave ig
Routing:
- net GND: track 570.1 -> 0.00 mm, vias 2 -> 0
- net VCC: track 459.9 -> 0.00 mm, vias 2 -> 0
- net ROW0: track 335.0 -> 0.00 mm, vias 2 -> 0
- net ROW2: track 326.8 -> 0.00 mm
- net ROW1: track 325.0 -> 0.00 mm
- net ROW4: track 263.9 -> 0.00 mm, vias 1 -> 0
- net COL0: track 262.9 -> 0.00 mm
- net COL1: track 248.5 -> 0.00 mm
- net ROW3: track 246.1 -> 0.00 mm, vias 1 -> 0
- net L_COL6: track 245.5 -> 0.00 mm, vias 1 -> 0
- net L_ROW4: track 245.1 -> 0.00 mm, vias 1 -> 0
- net L_ROW3: track 244.1 -> 0.00 mm, vias 1 -> 0
- net L_COL4: track 236.8 -> 0.00 mm, vias 1 -> 0
- net COL2: track 232.6 -> 0.00 mm
- net L_ROW1: track 226.8 -> 0.00 mm, vias 1 -> 0
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