File: pro micro version/pro micro version new traces.kicad_pcb (KiCad board)
At the start: 2 copper layers, 385.8 x 100 mm, 166 parts, among them SW1 SW_PUSH, U1 ProMicro

Commit message: finalized pcb design
Routing:
- net ROW0: track 216.3 -> 177.8 mm
Other:
- board text added: "Designed by Vaibhav Srivastava"
- board text added: "U.S.K.B."
Changed lines of the file:
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@@
   (general
     (thickness 1.6)
-    (drawings 9)
-    (tracks 855)
+    (drawings 11)
+    (tracks 849)
     (zones 0)
     (modules 166)
@@
     )
   )
+  (gr_text U.S.K.B. (at 28.575 75.692 -90) (layer F.SilkS)
+    (effects (font (size 1.905 1.905) (thickness 0.3)))
+  )
+  (gr_text "Designed by Vaibhav Srivastava" (at 25.4 88.10625 -90) (layer F.SilkS)
+    (effects (font (size 1.5 1.5) (thickness 0.3)))
+  )
   (gr_line (start 19.05 26.9875) (end 400.05 26.9875) (layer Edge.Cuts) (width 0.05))
   (gr_line (start 19.05 127) (end 19.84375 127) (layer Edge.Cuts) (width 0.05))
@@
   (segment (start 344.327001 41.177001) (end 350.739501 41.177001) (width 0.254) (layer B.Cu) (net 19))
   (segment (start 350.739501 41.177001) (end 362.74375 53.18125) (width 0.254) (layer B.Cu) (net 19))
-  (segment (start 373.788399 53.135499) (end 376.985499 53.135499) (width 0.254) (layer B.Cu) (net 19))
-  (segment (start 373.742648 53.18125) (end 373.788399 53.135499) (width 0.254) (layer B.Cu) (net 19))
-  (segment (start 362.74375 53.18125) (end 373.742648 53.18125) (width 0.254) (layer B.Cu) (net 19))
-  (segment (start 397.841149 57.616749) (end 398.93015 58.70575) (width 0.254) (layer B.Cu) (net 19))
-  (segment (start 381.466749 57.616749) (end 397.841149 57.616749) (width 0.254) (layer B.Cu) (net 19))
-  (segment (start 376.985499 53.135499) (end 381.466749 57.616749) (width 0.254) (layer B.Cu) (net 19))
   (segment (start 343.088538 53.9125) (end 346.075 53.9125) (width 0.254) (layer B.Cu) (net 20))
   (segment (start 336.938538 60.0625) (end 343.088538 53.9125) (width 0.254) (layer B.Cu) (net 20))
