File: pro micro version/pro micro version new traces.sch (KiCad schematic (older format))
At the start: 166 parts, among them SW1 SW_PUSH, U1 ProMicro

Commit message: finalized traces
Connections:
- net L_ROW0: now also L_U1.8 (5/C6); no longer L_U1.12 (9/B5)
- net L_ROW1: now also L_U1.9 (6/D7); no longer L_U1.11 (8/B4)
- net L_ROW3: now also L_U1.11 (8/B4); no longer L_U1.9 (6/D7)
- net L_ROW4: now also L_U1.12 (9/B5); no longer L_U1.8 (5/C6)
- net ROW0: now also U1.8 (5/C6); no longer U1.12 (9/B5)
- net ROW1: now also U1.9 (6/D7); no longer U1.11 (8/B4)
- net ROW3: now also U1.11 (8/B4); no longer U1.9 (6/D7)
- net ROW4: now also U1.12 (9/B5); no longer U1.8 (5/C6)
- no-connect marks 0 -> 4
Changed lines of the file:
@@
 Text GLabel 1000 950  0    50   Input ~ 0
 L_ROT_B
+Text GLabel 1000 1650 0    50   Input ~ 0
+L_ROW1
+Text GLabel 1000 1750 0    50   Input ~ 0
+L_ROW2
+Text GLabel 1000 1850 0    50   Input ~ 0
+L_ROW3
 Text GLabel 2400 1950 2    50   Input ~ 0
 L_COL0
@@
 Text GLabel 6800 950  0    50   Input ~ 0
 ROT_B
+Text GLabel 6800 1550 0    50   Input ~ 0
+ROW0
+Text GLabel 6800 1650 0    50   Input ~ 0
+ROW1
+Text GLabel 6800 1750 0    50   Input ~ 0
+ROW2
+Text GLabel 6800 1850 0    50   Input ~ 0
+ROW3
+Text GLabel 6800 1950 0    50   Input ~ 0
+ROW4
 Text GLabel 8200 1250 2    50   Input ~ 0
 COL0
@@
 $EndComp
 Text GLabel 1000 1550 0    50   Input ~ 0
+L_ROW0
+Text GLabel 1000 1950 0    50   Input ~ 0
 L_ROW4
-Text GLabel 1000 1950 0    50   Input ~ 0
-L_ROW0
-Text GLabel 1000 1650 0    50   Input ~ 0
-L_ROW3
-Text GLabel 1000 1750 0    50   Input ~ 0
-L_ROW2
-Text GLabel 1000 1850 0    50   Input ~ 0
-L_ROW1
-Text GLabel 6800 1550 0    50   Input ~ 0
-ROW4
-Text GLabel 6800 1650 0    50   Input ~ 0
-ROW3
-Text GLabel 6800 1750 0    50   Input ~ 0
-ROW2
-Text GLabel 6800 1850 0    50   Input ~ 0
-ROW1
-Text GLabel 6800 1950 0    50   Input ~ 0
-ROW0
+NoConn ~ 1000 1450
+NoConn ~ 2400 850
+NoConn ~ 6800 1450
+NoConn ~ 8200 850
+Text GLabel 3550 1450 0    50   Input ~ 0
+L_K_ENC
+Text GLabel 9300 1350 0    50   Input ~ 0
+K_ENC
 $EndSCHEMATC
