File: final/USKB Final.kicad_pcb (KiCad board)
At the start: 2 copper layers, 385.8 x 100 mm, 166 parts, among them SW1 SW_PUSH, U1 ProMicro

Commit message: finalized pcb design
Other:
- board text added: "U.S.K.B."
Changed lines of the file:
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@@
     )
   )
-  (gr_text "Designed by Vaibhav Srivastava" (at 28.575 88.10625 -90) (layer F.SilkS)
-    (effects (font (size 1.5 1.5) (thickness 0.3)))
+  (gr_text U.S.K.B. (at 28.575 75.692 -90) (layer F.SilkS)
+    (effects (font (size 1.905 1.905) (thickness 0.3)))
   )
   (gr_text "Designed by Vaibhav Srivastava" (at 25.4 88.10625 -90) (layer F.SilkS)
