File: final/USKB Final.sch (KiCad schematic (older format))
At the start: 166 parts, among them SW1 SW_PUSH, U1 ProMicro

Commit message: organized and exported files
Other:
- note added: "2"
- note added: "3/12/2021"
- note added: "U.S.K.B."
- note added: "unsplit keyboard"
Changed lines of the file:
@@
 	1    0    0    -1
 $EndComp
+Text Notes 12160 10960 0    98   ~ 20
+U.S.K.B.
+Text Notes 15390 11070 0    59   ~ 0
+2
+Text Notes 12220 10670 0    50   ~ 0
+unsplit keyboard
+Text Notes 12950 11070 0    50   ~ 0
+3/12/2021
 $EndSCHEMATC
