File: final/pcb and schema files/USKB Final.kicad_pcb (KiCad board)
At the start: 2 copper layers, 385.8 x 101.6 mm, 166 parts, among them SW1 SW_PUSH, U1 ProMicro

Commit message: changed bottom row to be more accessible
Parts:
- K_Space_2: footprint Keyboard Master List:MX-2.25U -> Keyboard Master List:MX-2.75U
- K_Space_3: footprint Keyboard Master List:MX-1.75U -> Keyboard Master List:MX-1.25U
- moved D_Space_2 5.56 mm to (192.1, 112.7)
- moved D_Space_3 5.56 mm to (230.2, 112.7)
- moved K_Space_3 4.76 mm to (221.5, 112.7)
- moved D_Caps1 4.76 mm to (91.3, 74.6)
- moved K_Space_2 4.76 mm to (183.4, 112.7)
Routing:
- net COL3: track 219.1 -> 226.2 mm
- net COL4: track 201.1 -> 206.9 mm
- net ROW4: track 263.2 -> 257.6 mm
- net L_ROW4: track 240.5 -> 246.0 mm
- net COL0: track 270.7 -> 275.7 mm
- net COL5: track 188.8 -> 193.0 mm
- net L_COL4: track 209.3 -> 212.7 mm
- net COL6: track 141.7 -> 138.7 mm
- net COL1: track 255.5 -> 258.1 mm
- net L_RESET: track 82.2 -> 83.7 mm
- net Net-(D_Space_2-Pad2): track 13.0 -> 14.1 mm
- net Net-(D_Caps1-Pad2): track 12.2 -> 13.2 mm
- net Net-(D_Space_3-Pad2): track 13.0 -> 13.9 mm
- net COL2: track 237.4 -> 238.1 mm
- net L_COL7: track 191.3 -> 190.8 mm

Commit message: changed smt lol
Other:
- board text added: "Designed by feynmantf"
- board text removed: "Designed by Vaibhav Srivastava"
