File: early revisions/bad wirings/wires are crazy im going to start moving stuff lol.kicad_pcb (KiCad board)
At the start: 2 copper layers, 338.1 x 104.8 mm, 163 parts, among them SW1 SW_PUSH, U1 ATmega32U4-AU, X1 XTAL_GND

Commit message: everything but simulation done
Parts:
- USB1: footprint Keebio Parts:HRO-TYPE-C-31-M-12-Assembly -> Keebio Parts:USB-C-12-Pin-MidMount
- moved C11 23.7 mm to (346.5, 36.1), turned to 270 degrees
- moved ENC1 15.8 mm to (332.2, 23.0), turned to 0 degrees
- moved C8 15.7 mm to (332.2, 59.4), turned to 180 degrees
- moved R7 14.1 mm to (333.0, 36.1)
- moved C4 12.3 mm to (332.2, 61.8), turned to 180 degrees
- moved R1 11.1 mm to (340.0, 72.0), turned to 0 degrees
- moved C3 9.15 mm to (344.3, 25.7), turned to 90 degrees
- moved C5 8.36 mm to (332.2, 64.6), turned to 180 degrees
- moved C9 8.06 mm to (336.3, 23.4), turned to 270 degrees
- moved C10 7.60 mm to (336.3, 27.1), turned to 90 degrees
- moved C1 5.85 mm to (338.7, 59.1)
- moved C2 5.85 mm to (341.0, 59.1)
- moved X1 5.85 mm to (339.9, 62.9)
- moved R5 4.84 mm to (338.7, 23.3), turned to 90 degrees
- moved C6 4.67 mm to (332.2, 67.3), turned to 180 degrees
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Routing:
- net GND: track 727.5 -> 522.5 mm, vias 1 -> 8
- net D-: track 463.2 -> 351.7 mm, vias 2 -> 0
- net D+: track 461.9 -> 356.7 mm, vias 2 -> 0
- net (no net): track 0.00 -> 84.2 mm
- net VCC: track 433.0 -> 502.4 mm, vias 2 -> 4
- net COL1: track 403.7 -> 446.4 mm, vias 4 -> 3
- net COL3: track 370.6 -> 407.9 mm, vias 2 -> 1
- net XTAL2: track 39.9 -> 10.2 mm, vias 2 -> 0
- net COL7: track 267.1 -> 296.7 mm, vias 2 -> 1
- net COL5: track 333.6 -> 304.6 mm, vias 2 -> 1
- net COL2: track 370.7 -> 399.2 mm, vias 2 -> 1
- net XTAL1: track 37.9 -> 9.80 mm, vias 2 -> 0
- net COL6: track 331.6 -> 306.3 mm, vias 2 -> 1
- net COL0: track 445.8 -> 470.7 mm, vias 4 -> 3
- net COL8: track 241.9 -> 259.7 mm, vias 2 -> 1
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Other:
- board text removed: "JLCJLCJLCJLC"
- board text removed: "U.S.K.B Designed by Feynman"
