File: final/pcb/unsplit-keyboard.kicad_pcb (KiCad board)
At the start: 2 copper layers, 338.1 x 104.8 mm, 163 parts, among them SW1 SW_PUSH, U1 ATmega32U4-AU, X1 XTAL_GND

Commit message: updated gerbers and all that
Other:
- board text added: "U.S.K.B Designed by V.S."
- board text removed: "U.S.K.B Designed by Feynman"
