File: final/pcb/kaluza.kicad_pcb (KiCad board)
At the start: 2 copper layers, 139 parts, among them SW1 Rotary_Encoder_Switch, U1 Elite-C

Commit message: update
Parts:
- added D_Spare: SMD_123, Keebio Parts:Diode-Hybrid-Back, F.Cu at (254.2, 9.62)
- added D_Spare: SMD_123, Keebio Parts:Diode-Hybrid-Back, F.Cu at (268.0, 9.62)
- added D_Spare: SMD_123, Keebio Parts:Diode-Hybrid-Back, F.Cu at (274.1, 2.03)
- added D_Spare: SMD_123, Keebio Parts:Diode-Hybrid-Back, F.Cu at (272.0, 4.57)
- added D_Spare: SMD_123, Keebio Parts:Diode-Hybrid-Back, F.Cu at (270.0, 7.11)
- added D_Spare: SMD_123, Keebio Parts:Diode-Hybrid-Back, F.Cu at (240.3, 9.62)
- added D_Spare: SMD_123, Keebio Parts:Diode-Hybrid-Back, F.Cu at (276.1, -0.51)
- moved D46 209.9 mm to (90.4, 7.08)
- moved D68 198.1 mm to (198.9, 9.62)
- moved D16 196.3 mm to (80.6, 2.00)
- moved D48 193.9 mm to (118.0, 7.08)
- moved D49 188.0 mm to (131.8, 7.08)
- moved D1 185.5 mm to (82.7, -0.54)
- moved D47 185.2 mm to (104.2, 7.08)
- moved D3 184.9 mm to (110.3, -0.54)
- moved D50 183.0 mm to (145.6, 7.08)
- moved D4 177.8 mm to (124.1, -0.54)
- moved D67 174.5 mm to (185.1, 9.62)
- moved D62 173.5 mm to (116.0, 9.62)
- moved D5 171.6 mm to (137.9, -0.54)
- moved D58 166.3 mm to (256.2, 7.08)
- moved D43 159.4 mm to (244.4, 4.54)
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
Commit message: idk what changed
Routing:
- net COL_6: track 0.00 -> 562.8 mm, vias 0 -> 2
- net COL_9: track 0.00 -> 522.0 mm, vias 0 -> 2
- net COL_7: track 0.00 -> 512.3 mm, vias 0 -> 2
- net COL_10: track 0.00 -> 494.9 mm, vias 0 -> 2
- net COL_8: track 0.00 -> 489.2 mm, vias 0 -> 2
- net COL_11: track 0.00 -> 485.3 mm, vias 0 -> 2
- net COL_12: track 0.00 -> 474.9 mm, vias 0 -> 2
- net COL_13: track 0.00 -> 431.2 mm, vias 0 -> 2
- net COL_14: track 0.00 -> 381.8 mm
- net ROT_A: track 0.00 -> 324.4 mm
- net ROT_B: track 0.00 -> 318.4 mm
- net ROW3: track 0.00 -> 300.8 mm, vias 0 -> 1
- net ROW0: track 0.00 -> 255.6 mm, vias 0 -> 1
- net ROW1: track 0.00 -> 249.9 mm, vias 0 -> 1
- net Net-(D15-Pad2): track 0.00 -> 245.3 mm
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